Commit message: added Magazin Dummy

File: fleximon/fleximon_data/data/magazin.urdf.xacro (robot description, xacro)
@@ -13,13 +13,13 @@
 		  <visual>
 		    <geometry>
-		      <mesh filename="package://fleximon_data/data/magazin.dae"/>
+		      <mesh filename="package://fleximon_data/data/Magazin_Dummy_M2.dae"/>
 		    </geometry>
-		    <origin rpy="0.0 0.0 0.0" xyz="0.39 -0.095 0.0"/>
+		    <origin rpy="0.0 0.0 0.0" xyz="0.030 -0.035 0.0"/>
 		  </visual>
 		  <collision>
 		    <geometry>
-		      <mesh filename="package://fleximon_data/data/magazin.dae"/>
+		      <mesh filename="package://fleximon_data/data/Magazin_Dummy_M2.dae"/>
 		    </geometry>
-		    <origin rpy="0.0 0.0 0.0" xyz="0.39 -0.095 0.0"/>
+		    <origin rpy="0.0 0.0 0.0" xyz="0.030 -0.035 0.0"/>
 		  </collision>
 		  <inertial>

File: fleximon/fleximon_data/data/ur5_fleximon.urdf.xacro (robot description, xacro)
@@ -18,6 +18,6 @@
   <!-- CALIBRATION -->
 	<!-- robot calibration | position of the robot relative to base link -->
-	<property name="arm_x" value="0.170"/>
-	<property name="arm_y" value="0.5825"/>
+	<property name="arm_x" value="0.3"/>
+	<property name="arm_y" value="0.6875"/>
 	<property name="arm_z" value="0.01"/>
 	<property name="arm_roll" value="0.0"/>
@@ -42,7 +42,7 @@
   	</xacro:fleximon>
 	<!-- Magazin -->
-	<!--xacro:magazin name="" parent="base_link"-->
-    		<!--origin xyz="0 0 0" rpy="0 0 0" /-->
-  	<!--/xacro:magazin-->
+	<xacro:magazin name="" parent="base_link">
+    		<origin xyz="0 0 0" rpy="0 0 0" />
+  	</xacro:magazin>
 <!-- Werkstuecktraeger -->
 	<!--xacro:werkstuecktraeger name="" parent="base_link"-->
