Commit message: TCP Tool changed and TeachIn status

File: fleximon/fleximon_data/data/ur5_fleximon.urdf.xacro (robot description, xacro)
@@ -11,5 +11,5 @@
 	<xacro:include filename="fleximon.urdf.xacro" />
 	<!-- environment model -->
-	<xacro:include filename="magazin.urdf.xacro" />
+	<!--xacro:include filename="magazin.urdf.xacro" /-->
 	<!-- environment model -->
 	<!--xacro:include filename="werkstuecktraeger.urdf.xacro" /-->
@@ -18,6 +18,6 @@
   <!-- CALIBRATION -->
 	<!-- robot calibration | position of the robot relative to base link -->
-	<property name="arm_x" value="0.3"/>
-	<property name="arm_y" value="0.6875"/>
+	<property name="arm_x" value="0.335"/>
+	<property name="arm_y" value="0.5875"/>
 	<property name="arm_z" value="0.01"/>
 	<property name="arm_roll" value="0.0"/>
@@ -52,5 +52,5 @@
 	<xacro:afag_gripper name="${arm_prefix}" parent="${arm_prefix}ee_link">
     		<!-- gripper offset -->
-				<origin xyz="0 0 0" rpy="0 0 0" />
+				<origin xyz="0.104 0 0" rpy="-0.785 0 0" />
 		</xacro:afag_gripper>
 	<joint name="{arm_prefix}ee_joint" type="fixed" >
